File: Nixie Clock ECE5930/Nixie Clock ECE5930.kicad_pcb (KiCad board)
At the start: 2 copper layers, 217.4 x 43.5 mm, 44 parts, among them J1 Conn_02x03_Top_Bottom, J2 PJ-002B, J3 Conn_01x03, SW4 2-1825910-7, SW5 2-1825910-7, SW6 2-1825910-7, U1 ATmega328P-P, U2 HV5622, U3 HV5622, U4 L78L05_SO8, U5 DS3231N, U6 L78L05_SOT89

Commit message: final build maybe?
Parts:
- removed BT1: Battery, Battery:Battery_Panasonic_CR2032-HFN_Horizontal_CircularHoles
- added BT2: BC-2600, BC_2600_TR (1):BAT_BC-2600, F.Cu at (41.0, 43.8)
- C4, C5: value C -> 0.1uF
- U2: footprint HV5622PG-G:QFP80P1390X1390X235-44N -> KiCad:QFP80P1390X1390X235-44N
Connections:
- R10 pad 1: Net-(N5-PadA) -> Net-(R10-Pad1)
- R11 pad 2: Net-(N8-PadA) -> Net-(R11-Pad2)
- R4 pad 1: Net-(N4-PadA) -> Net-(R4-Pad1)
- R5 pad 1: Net-(N3-PadA) -> Net-(R5-Pad1)
- R6 pad 1: Net-(N2-PadA) -> Net-(R6-Pad1)
- R7 pad 1: Net-(N1-PadA) -> Net-(R7-Pad1)
- R8 pad 1: Net-(N7-PadA) -> Net-(R8-Pad1)
- R9 pad 1: Net-(N6-PadA) -> Net-(R9-Pad1)
Routing:
- net Net-(U5-Vbat): track 50.7 -> 92.0 mm, vias 3 -> 1
- net +5V: track 474.9 -> 489.1 mm, vias 11 -> 10
