File: Nixie Clock ECE5930/Nixie Clock ECE5930.kicad_sch (KiCad schematic)
At the start: 37 parts, among them J1 Conn_02x03_Top_Bottom, J2 USB_C_Receptacle_PowerOnly_6P, J3 Conn_01x03, SW1 SW_Push, SW2 SW_Push, SW3 SW_Push, U1 ATmega328P-P, U2 HV5622, U3 HV5622, U4 L78L05_SO8, U5 DS3231N, Y1 Crystal

Commit message: added button STEP
Parts:
- removed J2: USB_C_Receptacle_PowerOnly_6P, Connector_USB:USB_C_Plug_JAE_DX07P024AJ1, symbol Connector:USB_C_Receptacle_PowerOnly_6P
- removed SW1, SW2, SW3: SW_Push, Button_Switch_SMD:Nidec_Copal_CAS-120A, symbol Switch:SW_Push
- added SW4, SW5, SW6: 2-1825910-7, SW4_1825910-G_TEC, symbol switch4:2-1825910-7
Connections:
- net +5V: now also SW4.3, SW4.4, SW5.3, SW5.4, SW6.3, SW6.4
- net at U1.13 (PD7): now also SW6.1, SW6.2
- net at U1.12 (PD6): now also SW5.1, SW5.2
- net at U1.11 (PD5): now also SW4.1, SW4.2

Commit message: holy shit im gonna die
Parts:
- removed C4, C5: 0.1uF, Capacitor_SMD:C_2220_5750Metric, symbol Device:C
- removed U4: L78L05_SO8, Package_SO:SOIC-8_3.9x4.9mm_P1.27mm, symbol Regulator_Linear:L78L05_SO8
- added J2: PJ-002B, PJ-002B:CUI_PJ-002B, symbol PJ-002B:PJ-002B
Connections:
- net +12V: now also J2.1
- net +5V: now also J2.2, J2.3

Commit message: 3d models yum
Parts:
- J2: footprint PJ-002B:CUI_PJ-002B -> PJ_002B:CUI_PJ-002B
- SW4, SW5, SW6: footprint SW4_1825910-G_TEC -> footprints:SW4_1825910-G_TEC
- U3: footprint HV5622PG-G:QFP80P1390X1390X235-44N -> KiCad:QFP80P1390X1390X235-44N
Changed lines of the file:
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@@
 			)
 		)
-		(property "Footprint" "SW4_1825910-G_TEC"
+		(property "Footprint" "footprints:SW4_1825910-G_TEC"
 			(at 120.65 261.62 0)
 			(effects
@@
 			)
 		)
-		(property "Footprint" "SW4_1825910-G_TEC"
+		(property "Footprint" "footprints:SW4_1825910-G_TEC"
 			(at 120.65 236.22 0)
 			(effects
@@
 			)
 		)
-		(property "Footprint" "HV5622PG-G:QFP80P1390X1390X235-44N"
+		(property "Footprint" "KiCad:QFP80P1390X1390X235-44N"
 			(at 340.36 93.98 0)
 			(effects
@@
 			)
 		)
-		(property "Footprint" "SW4_1825910-G_TEC"
+		(property "Footprint" "footprints:SW4_1825910-G_TEC"
 			(at 119.38 210.82 0)
 			(effects
@@
 	)
 	(symbol
+		(lib_name "HV5622_1")
 		(lib_id "nixie-cache:HV5622")
 		(at 340.36 220.98 0)
@@
 			)
 		)
-		(property "Footprint" "PJ-002B:CUI_PJ-002B"
+		(property "Footprint" "PJ_002B:CUI_PJ-002B"
 			(at 185.42 313.69 0)
 			(effects

Commit message: final commit i hope
Parts:
- removed Y1: Crystal, nixiemisc:nixiemisc-CRYSTAL-SMD-2.0X1.6MM, symbol Device:Crystal
- added C4, C5: C, Capacitor_SMD:C_2220_5750Metric, symbol Device:C
- added C6: ABS07-32.768KHZ-T, ABS07_32_768KHZ_T (1):CAP_ABS07-32.768KHZ-T_ABR, symbol 2025-11-13_06-06-08:ABS07-32.768KHZ-T
- added U6: L78L05_SOT89, Package_TO_SOT_SMD:SOT-89-3, symbol Regulator_Linear:L78L05_SOT89
Connections:
- net +12V: now also U6.3 (IN)
- net +5V: now also C4.1, C4.2, C5.1, C5.2, U6.1 (OUT), U6.2 (GND)
- net at C3.2, U1.10 (XTAL2/PB7): now also C6.1
- net at C2.1, U1.9 (XTAL1/PB6): now also C6.2
Other:
- moved on the sheet: J2, J3

Commit message: final build maybe?
Parts:
- removed BT1: Battery, Battery:Battery_Panasonic_CR2032-HFN_Horizontal_CircularHoles, symbol nixie-cache:Battery
- added BT2: BC-2600, BC_2600_TR (1):BAT_BC-2600, symbol BC-2600:BC-2600
- C1: MFR (Manufacturer) (none) -> Walsin Technology Corporation; MPN (Manufacturer Part Number) (none) -> 0402B104K160CT; SPN (Supplier Part Number) (none) -> 1292-1630-2-ND - Tape & Reel (TR); SPR (Supplier) (none) -> DigiKey
- C2, C3: MFR (Manufacturer) (none) -> KEMET; MPN (Manufacturer Part Number) (none) -> C0603C220J5GACTU; SPN (Supplier Part Number) (none) -> C0603C220J5GACTU; SPR (Supplier) (none) -> DigiKey
- C4, C5: value C -> 0.1uF; MFR (Manufacturer) (none) -> Walsin Technology Corporation; MPN (Manufacturer Part Number) (none) -> 0402B104K160CT; SPN (Supplier Part Number) (none) -> 1292-1630-2-ND - Tape & Reel (TR); SPR (Supplier) (none) -> DigiKey
- C6: MFR (Manufacturer) (none) -> Abracon LLC; MPN (Manufacturer Part Number) (none) -> ABS07-32.768KHZ-T; SPN (Supplier Part Number) (none) -> 535-9542-2-ND - Tape & Reel (TR); SPR (Supplier) (none) -> DigiKey
- J1: MFR (Manufacturer) (none) -> Amphenol ICC (FCI); MPN (Manufacturer Part Number) (none) -> 10125394-T0803ALF; SPN (Supplier Part Number) (none) -> 609-10125394-T0803ALFTR-ND - Tape & Reel (TR); SPR (Supplier) (none) -> DigiKey
- J2: MANUFACTURER CUI INC -> (none); MFR (Manufacturer) (none) -> Same Sky (Formerly CUI Devices); MPN (Manufacturer Part Number) (none) -> PJ-002B; SPN (Supplier Part Number) (none) -> CP-002B-ND; SPR (Supplier) (none) -> DigiKey
- J3: MFR (Manufacturer) (none) -> Amphenol ICC (Commercial Products); MPN (Manufacturer Part Number) (none) -> G800W305018EU; SPN (Supplier Part Number) (none) -> 664-G800W305018EU-ND; SPR (Supplier) (none) -> DigiKey
- N1, N2, N3, N5, N6, N7: value ~ -> IN-14; MPN (Manufacturer Part Number) (none) -> ${ITEM_NUMBER}; now not fitted; now left out of the parts list
- N4, N8: MPN (Manufacturer Part Number) (none) -> ${ITEM_NUMBER}; now not fitted; now left out of the parts list
- R1: MFR (Manufacturer) (none) -> YAGEO; MPN (Manufacturer Part Number) (none) -> RC0603FR-0710KL; SPN (Supplier Part Number) (none) -> 311-10.0KHRTR-ND - Tape & Reel (TR); SPR (Supplier) (none) -> DigiKey
- R10, R5, R6, R7, R8, R9: MFR (Manufacturer) (none) -> RMCF0603FT27K4TR-ND - Tape & Reel (TR); MPN (Manufacturer Part Number) (none) -> RMCF0603FT27K4; SPN (Supplier Part Number) (none) -> Stackpole Electronics Inc; SPR (Supplier) (none) -> DigiKey
- R11, R4: MFR (Manufacturer) (none) -> YAGEO; MPN (Manufacturer Part Number) (none) -> RC0402FR-07100KL; SPN (Supplier Part Number) (none) -> 311-100KLRTR-ND - Tape & Reel (TR); SPR (Supplier) (none) -> DigiKey
- R2, R3: MFR (Manufacturer) (none) -> Vishay Dale; MPN (Manufacturer Part Number) (none) -> CRCW08057K00JNTA; SPN (Supplier Part Number) (none) -> CRCW08057K00JNTA-ND - Tape & Reel (TR); SPR (Supplier) (none) -> DigiKey
- SW4, SW5, SW6: MFR (Manufacturer) (none) -> TE Connectivity ALCOSWITCH Switches; MPN (Manufacturer Part Number) (none) -> RMCF0603FT27K4; SPN (Supplier Part Number) (none) -> 450-1653-ND; SPR (Supplier) (none) -> DigiKey
- U1: MFR (Manufacturer) (none) -> Microchip Technology; MPN (Manufacturer Part Number) (none) -> ATMEGA328P-PU; SPN (Supplier Part Number) (none) -> ATMEGA328P-PU-ND; SPR (Supplier) (none) -> DigiKey
- U2: footprint HV5622PG-G:QFP80P1390X1390X235-44N -> KiCad:QFP80P1390X1390X235-44N; MFR (Manufacturer) (none) -> Microchip Technology; MPN (Manufacturer Part Number) (none) -> HV5622PG-G; SPN (Supplier Part Number) (none) -> HV5622PG-G-ND; SPR (Supplier) (none) -> DigiKey
- U3: MFR (Manufacturer) (none) -> Microchip Technology; MPN (Manufacturer Part Number) (none) -> HV5622PG-G; SPN (Supplier Part Number) (none) -> HV5622PG-G-ND; SPR (Supplier) (none) -> DigiKey
- U4: renamed from U6; MFR (Manufacturer) (none) -> UMW; MPN (Manufacturer Part Number) (none) -> 78L05; SPN (Supplier Part Number) (none) -> 4518-78L05TR-ND; SPR (Supplier) (none) -> DigiKey
- U5: MFR (Manufacturer) (none) -> Analog Devices Inc./Maxim Integrated; MPN (Manufacturer Part Number) (none) -> DS3231S#T&R; SPN (Supplier Part Number) (none) -> DS3231S#T&RTR-ND; SPR (Supplier) (none) -> DigiKey
Connections:
- net +5V: now also BT2.1, BT2.2
- net at U5.14 (Vbat): now also BT2.S1, BT2.S2, BT2.S3
- no-connect marks 0 -> 1
Other:
- note added: "Bobby Thompson"
